File: surface-mount/cvbs-oscilloscope-meter.kicad_sch (KiCad schematic)
At the start: 38 parts, among them J1 Conn_Coaxial_Power, J2 Conn_Coaxial_Power, J3 Conn_Coaxial_Power, J4 Conn_Coaxial_Power, Q1 2N3906, Q2 2N3906, Q3 2N3904, Q4 2N3904, Q5 2N3904, Q6 2N3904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

Commit message: Created SMD boards
Parts:
- removed U3: AD8032_B, Package_DIP:DIP-8_W7.62mm_Socket_LongPads, symbol Device:Opamp_Dual
- removed U4: AD8032, Package_DIP:DIP-8_W7.62mm_Socket_LongPads, symbol Device:Opamp_Dual
- added D3: Indicator, LED_SMD:LED_0805_2012Metric_Pad1.15x1.40mm_HandSolder, symbol Device:LED_Filled
- added J5: Conn_01x02, Connector_Molex:Molex_KK-396_A-41791-0002_1x02_P3.96mm_Vertical, symbol Connector_Generic:Conn_01x02
- added J6: Conn_01x02, Connector_BarrelJack:BarrelJack_CUI_PJ-063AH_Horizontal, symbol Connector_Generic:Conn_01x02
- added MK1, MK2, MK3, MK4: MountingHole_Pad, Mounting_Holes:MountingHole_3.2mm_M3_ISO7380, symbol Mechanical:MountingHole_Pad
- added R16: 2.4k, Resistor_SMD:R_0805_2012Metric_Pad1.20x1.40mm_HandSolder, symbol Device:R_US
- added unit 2 of U2
- added unit 3 of U2
- C1: value 100n -> 0.1u; footprint Capacitor_THT:C_Disc_D7.5mm_W2.5mm_P5.00mm -> Capacitor_SMD:C_0805_2012Metric_Pad1.18x1.45mm_HandSolder
- C2, C3, C4, C5: footprint Capacitor_THT:C_Disc_D7.5mm_W2.5mm_P5.00mm -> Capacitor_SMD:C_0805_2012Metric_Pad1.18x1.45mm_HandSolder
- D1, D2: footprint Diode_THT:D_DO-35_SOD27_P7.62mm_Horizontal -> Diode_SMD:D_SOD-123
- Q1, Q2, Q3, Q4, Q5, Q6: footprint Package_TO_SOT_THT:TO-92_Inline -> Package_TO_SOT_SMD:SOT-23
- R1, R10, R11, R12, R13, R14, R15, R2, R3, R4, R5, R6, R7, R8, R9: footprint Resistor_THT:R_Axial_DIN0207_L6.3mm_D2.5mm_P10.16mm_Horizontal -> Resistor_SMD:R_0805_2012Metric_Pad1.20x1.40mm_HandSolder
- RV1, RV2: footprint Resistor_THT:R_Axial_DIN0207_L6.3mm_D2.5mm_P10.16mm_Horizontal -> Potentiometer_THT:Potentiometer_Piher_PC-16_Single_Vertical
- U1: footprint Package_DIP:DIP-8_W7.62mm_Socket_LongPads -> Package_SO:SOIC-8_3.9x4.9mm_P1.27mm
- U2: value AD8032_A -> AD8032; footprint Package_DIP:DIP-8_W7.62mm_Socket_LongPads -> Package_SO:SOIC-8_3.9x4.9mm_P1.27mm
Connections:
- net +9V: now also D3.2 (A), J5.1 (Pin_1), J6.1 (Pin_1), U2.8 (V+)
- net GND: now also J5.2 (Pin_2), J6.2 (Pin_2), R16.2, U2.4 (V-)
- net at U2.3 (+): now also U2.6 (-), U2.7
- net at RV2.2: now also U2.5 (+)
- new net: D3.1 (K), R16.1
- no-connect marks 2 -> 6
