File: tht/cvbs-oscilloscope-meter-rounded.kicad_pcb (KiCad board)
At the start: 2 copper layers, 52.2 x 113.8 mm, 50 parts, among them J1 Conn_Coaxial_Power, J2 Conn_Coaxial_Power, J3 Conn_Coaxial_Power, J4 Conn_Coaxial_Power, J5 Barrel_Jack_Switch, J6 Molex 3.96mm, Q1 2N3906, Q2 2N3906, Q3 2N3904, Q4 2N3904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

Commit message: Updated routing
Updated routing
Parts:
- added REF** (x2): OSHW-Logo_7.5x8mm_Copper, Symbol:OSHW-Logo_7.5x8mm_Copper, F.Cu at (107.8, 171.1)
